File: schematic/wiring.kicad_sch (KiCad schematic)
At the start: 4 parts, among them U1 DEVKIT_V1_ESP32-WROOM-32, U2 815

Commit message: pull up
Parts:
- added R2, R3: R4k7, symbol Device:R
Connections:
- net at U1.1 (3V3), U2.V+_1 (V+), U2.V+_10 (V+)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: now also R2.1, R3.1
- net at U1.18 (CMD), U2.SDA_1 (SDA), U2.SDA_2 (SDA): now also R2.2
- net at U1.19 (EXT_5V), U2.SCL_1 (SCL), U2.SCL_2 (SCL): now also R3.2
Changed lines of the file:
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@@
 (kicad_sch (version 20230121) (generator eeschema)
   (paper "A4")
+  (junction (at 91.44 40.64) (diameter 0) (color 0 0 0 0)
+  )
+  (junction (at 63.5 40.64) (diameter 0) (color 0 0 0 0)
+  )
   (junction (at 135.89 125.73) (diameter 0) (color 0 0 0 0)
   )
   (junction (at 144.78 176.53) (diameter 0) (color 0 0 0 0)
   )
+  (junction (at 54.61 95.25) (diameter 0) (color 0 0 0 0)
+  )
+  (junction (at 63.5 97.79) (diameter 0) (color 0 0 0 0)
+  )
   (wire (pts (xy 158.75 40.64) (xy 91.44 40.64))
     (stroke (width 0) (type default))
   )
-  (wire (pts (xy 58.42 97.79) (xy 97.79 97.79))
+  (wire (pts (xy 58.42 97.79) (xy 63.5 97.79))
     (stroke (width 0) (type default))
   )
@@
     (stroke (width 0) (type default))
   )
+  (wire (pts (xy 54.61 40.64) (xy 63.5 40.64))
+    (stroke (width 0) (type default))
+  )
   (wire (pts (xy 135.89 133.35) (xy 144.78 133.35))
     (stroke (width 0) (type default))
@@
     (stroke (width 0) (type default))
   )
+  (wire (pts (xy 63.5 69.85) (xy 63.5 40.64))
+    (stroke (width 0) (type default))
+  )
+  (wire (pts (xy 63.5 77.47) (xy 63.5 97.79))
+    (stroke (width 0) (type default))
+  )
+  (wire (pts (xy 54.61 77.47) (xy 54.61 95.25))
+    (stroke (width 0) (type default))
+  )
   (wire (pts (xy 135.89 176.53) (xy 144.78 176.53))
     (stroke (width 0) (type default))
@@
     (stroke (width 0) (type default))
   )
+  (wire (pts (xy 63.5 97.79) (xy 97.79 97.79))
+    (stroke (width 0) (type default))
+  )
   (wire (pts (xy 144.78 140.97) (xy 144.78 152.4))
     (stroke (width 0) (type default))
@@
     (stroke (width 0) (type default))
   )
+  (wire (pts (xy 63.5 40.64) (xy 91.44 40.64))
+    (stroke (width 0) (type default))
+  )
   (wire (pts (xy 135.89 125.73) (xy 135.89 128.27))
     (stroke (width 0) (type default))
@@
   )
   (wire (pts (xy 158.75 125.73) (xy 158.75 40.64))
+    (stroke (width 0) (type default))
+  )
+  (wire (pts (xy 54.61 69.85) (xy 54.61 40.64))
     (stroke (width 0) (type default))
   )
@@
     )
   )
+  (symbol (lib_id "Device:R") (at 54.61 73.66 0) (unit 1)
+    (in_bom yes) (on_board yes) (dnp no) (fields_autoplaced)
+    (property "Reference" "R2" (at 57.15 72.39 0)
+      (effects (font (size 1.27 1.27)) (justify left))
+    )
+    (property "Value" "R4k7" (at 57.15 74.93 0)
+      (effects (font (size 1.27 1.27)) (justify left))
+    )
+    (property "Footprint" "" (at 52.832 73.66 90)
+      (effects (font (size 1.27 1.27)) hide)
+    )
+    (property "Datasheet" "~" (at 54.61 73.66 0)
+      (effects (font (size 1.27 1.27)) hide)
+    )
+    (pin "2")
+    (pin "1")
+    (instances
+      (project "wiring"
+        (path "/1b186eef-9e5f-4f3b-86cc-a2a2196dea3d"
+          (reference "R2") (unit 1)
+        )
+      )
+    )
+  )
   (symbol (lib_id "Device:R") (at 144.78 156.21 0) (unit 1)
     (in_bom yes) (on_board yes) (dnp no) (fields_autoplaced)
@@
         )
       )
+    )
+  )
+  (symbol (lib_id "Device:R") (at 63.5 73.66 0) (unit 1)
+    (in_bom yes) (on_board yes) (dnp no) (fields_autoplaced)
+    (property "Reference" "R3" (at 66.04 72.39 0)
+      (effects (font (size 1.27 1.27)) (justify left))
+    )
+    (property "Value" "R4k7" (at 66.04 74.93 0)
+      (effects (font (size 1.27 1.27)) (justify left))
+    )
+    (property "Footprint" "" (at 61.722 73.66 90)
+      (effects (font (size 1.27 1.27)) hide)
+    )
+    (property "Datasheet" "~" (at 63.5 73.66 0)
+      (effects (font (size 1.27 1.27)) hide)
+    )
+    (pin "2")
+    (pin "1")
+    (instances
+      (project "wiring"
+        (path "/1b186eef-9e5f-4f3b-86cc-a2a2196dea3d"
+          (reference "R3") (unit 1)
+        )
+      )
